File: CAD/processor.kicad_sch (KiCad schematic)
At the start: 0 parts

Commit message: Added processor symbol for STM32G473RCT6
Parts:
- added U1: STM32G473RCTx, Package_QFP:LQFP-64_10x10mm_P0.5mm, symbol MCU_ST_STM32G4:STM32G473RCTx
Connections:
- new net: U1.15 (VSS), U1.31 (VSS), U1.47 (VSS), U1.63 (VSS)
Changed lines of the file:
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@@
 	(generator_version "9.0")
 	(paper "A4")
+	(symbol
+		(lib_id "MCU_ST_STM32G4:STM32G473RCTx")
+		(at 132.08 93.98 0)
+		(unit 1)
+		(exclude_from_sim no)
+		(in_bom yes)
+		(on_board yes)
+		(dnp no)
+		(fields_autoplaced yes)
+		(property "Reference" "U1"
+			(at 136.7633 142.24 0)
+			(effects
+				(font
+					(size 1.27 1.27)
+				)
+				(justify left)
+			)
+		)
+		(property "Value" "STM32G473RCTx"
+			(at 136.7633 144.78 0)
+			(effects
+				(font
+					(size 1.27 1.27)
+				)
+				(justify left)
+			)
+		)
+		(property "Footprint" "Package_QFP:LQFP-64_10x10mm_P0.5mm"
+			(at 116.84 139.7 0)
+			(effects
+				(font
+					(size 1.27 1.27)
+				)
+				(justify right)
+				(hide yes)
+			)
+		)
+		(property "Datasheet" "https://www.st.com/resource/en/datasheet/stm32g473rc.pdf"
+			(at 132.08 93.98 0)
+			(effects
+				(font
+					(size 1.27 1.27)
+				)
+				(hide yes)
+			)
+		)
+		(property "Description" "STMicroelectronics Arm Cortex-M4 MCU, 256KB flash, 128KB RAM, 170 MHz, 1.71-3.6V, 52 GPIO, LQFP64"
+			(at 132.08 93.98 0)
+			(effects
+				(font
+					(size 1.27 1.27)
+				)
+				(hide yes)
+			)
+		)
+		(property "LCSC" "C529361"
+			(at 132.08 93.98 0)
+			(effects
+				(font
+					(size 1.27 1.27)
+				)
+				(hide yes)
+			)
+		)
+		(pin "12"
+		)
+		(pin "32"
+		)
+		(pin "59"
+		)
+		(pin "62"
+		)
+		(pin "57"
+		)
+		(pin "30"
+		)
+		(pin "61"
+		)
+		(pin "58"
+		)
+		(pin "60"
+		)
+		(pin "33"
+		)
+		(pin "27"
+		)
+		(pin "47"
+		)
+		(pin "31"
+		)
+		(pin "21"
+		)
+		(pin "20"
+		)
+		(pin "53"
+		)
+		(pin "4"
+		)
+		(pin "56"
+		)
+		(pin "15"
+		)
+		(pin "9"
+		)
+		(pin "10"
+		)
+		(pin "44"
+		)
+		(pin "42"
+		)
+		(pin "43"
+		)
+		(pin "41"
+		)
+		(pin "40"
+		)
+		(pin "63"
+		)
+		(pin "46"
+		)
+		(pin "34"
+		)
+		(pin "48"
+		)
+		(pin "35"
+		)
+		(pin "8"
+		)
+		(pin "13"
+		)
+		(pin "16"
+		)
+		(pin "51"
+		)
+		(pin "45"
+		)
+		(pin "36"
+		)
+		(pin "29"
+		)
+		(pin "26"
+		)
+		(pin "54"
+		)
+		(pin "2"
+		)
+		(pin "7"
+		)
+		(pin "5"
+		)
+		(pin "6"
+		)
+		(pin "55"
+		)
+		(pin "39"
+		)
+		(pin "3"
+		)
+		(pin "28"
+		)
+		(pin "23"
+		)
+		(pin "14"
+		)
+		(pin "49"
+		)
+		(pin "52"
+		)
+		(pin "11"
+		)
+		(pin "22"
+		)
+		(pin "37"
+		)
+		(pin "18"
+		)
+		(pin "1"
+		)
+		(pin "38"
+		)
+		(pin "19"
+		)
+		(pin "17"
+		)
+		(pin "25"
+		)
+		(pin "24"
+		)
+		(pin "50"
+		)
+		(pin "64"
+		)
+		(instances
+			(project "motherboard"
+				(path "/35ffd292-e089-4bd5-9273-a58251615447/c72d0478-d97d-47c0-92e8-6bb9c0fc8305"
+					(reference "U1")
+					(unit 1)
+				)
+			)
+		)
+	)
 )
